Commit message: [Update] リアルモデルに変更

File: Assets/URDF/mycobot_description/urdf/color.xacro (robot description, xacro)
@@ -13,3 +13,6 @@
     <color rgba="1.0 1.0 1.0 1.0" />
   </material>
+  <material name="gray">
+    <color rgba="0.9 0.9 0.9 1.0" />
+  </material>
 </robot>

File: Assets/URDF/mycobot_description/urdf/mycobot.urdf (robot description, URDF)
Before this commit: robot mycobot, 8 links, 7 joints
Links:
- added link world
- link base_link: mass None -> 1.0; geometry collision mesh filename=package://mycobot_description/meshes/stl/visual/base_link.s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 scale=0.001 0.001 0.001; visual mesh filename=package://mycobot_description/meshes/stl/visual/base_link.d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 scale=0.001 0.001 0.001
- link link1: mass None -> 1.0; geometry collision mesh filename=package://mycobot_description/meshes/stl/collision/link1.stl; visual mesh filename=package://mycobot_description/meshes/stl/visual/link1.dae
- link link2: mass None -> 0.2; geometry collision mesh filename=package://mycobot_description/meshes/stl/collision/link2.stl; visual mesh filename=package://mycobot_description/meshes/stl/visual/link2.dae
- link link3: mass None -> 0.4; geometry collision mesh filename=package://mycobot_description/meshes/stl/collision/link3.stl; visual mesh filename=package://mycobot_description/meshes/stl/visual/link3.dae
- link link4: mass None -> 0.4; geometry collision mesh filename=package://mycobot_description/meshes/stl/collision/link4.stl; visual mesh filename=package://mycobot_description/meshes/stl/visual/link4.dae
- link link5: mass None -> 0.2; geometry collision mesh filename=package://mycobot_description/meshes/stl/collision/link5.stl; visual mesh filename=package://mycobot_description/meshes/stl/visual/link5.dae
- link link6: mass None -> 0.5; geometry collision mesh filename=package://mycobot_description/meshes/stl/collision/link6.stl; visual mesh filename=package://mycobot_description/meshes/stl/visual/link6.dae
- link link6_flange: mass None -> 0.1; geometry collision mesh filename=package://mycobot_description/meshes/stl/collision/link7.stl; visual mesh filename=package://mycobot_description/meshes/stl/visual/link7.dae
Joints:
- added joint base_link_to_world_joint: type fixed, parent world, child base_link
- joint base_joint: origin xyz=0 0 0 rpy=0 0 1.57 -> xyz=0 0 0.006 rpy=0 0 1.570795
- joint joint1: limit lower=-3.14 upper=3.14159 effort=1000.0 velocity=0 -> lower=-3.14159 upper=3.14159 effort=10.0 velocity=1.0
- joint joint2: limit lower=-3.14 upper=3.14159 effort=1000.0 velocity=0 -> lower=-3.14159 upper=3.14159 effort=10.0 velocity=1.0
- joint joint3: limit lower=-3.14 upper=3.14159 effort=1000.0 velocity=0 -> lower=-3.14159 upper=3.14159 effort=10.0 velocity=1.0
- joint joint4: limit lower=-3.14 upper=3.14159 effort=1000.0 velocity=0 -> lower=-3.14159 upper=3.14159 effort=10.0 velocity=1.0
- joint joint5: limit lower=-3.14 upper=3.14159 effort=1000.0 velocity=0 -> lower=-3.14159 upper=3.14159 effort=10.0 velocity=1.0
- joint joint6: axis 0 1 0 -> 0 0 1; limit lower=-3.14 upper=3.14159 effort=1000.0 velocity=0 -> lower=-3.14159 upper=3.14159 effort=10.0 velocity=1.0; origin xyz=0 0.0456 0.03792 rpy=0 0 0 -> xyz=0 0.0351 0.03792 rpy=-1.570795 0 0

File: Assets/URDF/mycobot_description/urdf/mycobot.urdf.xacro (robot description, xacro)
@@ -15,10 +15,10 @@
     <child link="base_link" />
   </joint>
-  <link name="camera_link"/>
+  <!-- <link name="camera_link"/>
   <joint name="joint_kinect_first" type="fixed">
     <origin xyz="-0.7137 0.215 0.4331" rpy="-0.0415 0.3679 -0.2391" />
     <parent link="world"/>
     <child link="camera_link"/>
-  </joint>
+  </joint> -->
   <!-- <joint name="joint_rgb_kinect_first" type="fixed">
     <origin rpy="${M_PI/2} ${M_PI} ${M_PI/2}"/>
@@ -35,5 +35,5 @@
       <visual>
         <geometry>
-          <mesh filename="package://mycobot_description/meshes/stl/visual/base_link.stl" scale="0.001 0.001 0.001" />
+          <mesh filename="package://mycobot_description/meshes/stl/visual/base_link.dae" scale="0.001 0.001 0.001" />
         </geometry>
         <origin xyz="0 0 0" rpy="0 0 ${M_PI}" />

File: Assets/URDF/mycobot_description/urdf/mycobot.xacro (robot description, xacro)
@@ -26,5 +26,5 @@
       <visual>
         <geometry>
-          <mesh filename="package://mycobot_description/meshes/stl/visual/link1.stl" />
+          <mesh filename="package://mycobot_description/meshes/stl/visual/link1.dae" />
         </geometry>
         <origin xyz="0 0 0" rpy="0 0 0" />
@@ -34,4 +34,5 @@
         <geometry>
           <mesh filename="package://mycobot_description/meshes/stl/collision/link1.stl" />
+          <!-- <mesh filename="package://mycobot_description/meshes/stl/visual/link1.stl" /> -->
         </geometry>
         <origin xyz="0 0 0" rpy="0 0 0" />
@@ -46,5 +47,5 @@
       <visual>
         <geometry>
-          <mesh filename="package://mycobot_description/meshes/stl/visual/link2.stl" />
+          <mesh filename="package://mycobot_description/meshes/stl/visual/link2.dae" />
         </geometry>
         <origin xyz="0 0 0" rpy="0 0 0" />
@@ -54,4 +55,5 @@
         <geometry>
           <mesh filename="package://mycobot_description/meshes/stl/collision/link2.stl" />
+          <!-- <mesh filename="package://mycobot_description/meshes/stl/visual/link2.stl" /> -->
         </geometry>
         <origin xyz="0 0 0" rpy="0 0 0" />
@@ -66,5 +68,5 @@
       <visual>
         <geometry>
-          <mesh filename="package://mycobot_description/meshes/stl/visual/link3.stl" />
+          <mesh filename="package://mycobot_description/meshes/stl/visual/link3.dae" />
         </geometry>
         <origin xyz="0 0 0" rpy="0 0 0" />
@@ -74,4 +76,5 @@
         <geometry>
           <mesh filename="package://mycobot_description/meshes/stl/collision/link3.stl" />
+          <!-- <mesh filename="package://mycobot_description/meshes/stl/visual/link3.stl" /> -->
         </geometry>
         <origin xyz="0 0 0" rpy="0 0 0" />
@@ -86,5 +89,5 @@
       <visual>
         <geometry>
-          <mesh filename="package://mycobot_description/meshes/stl/visual/link4.stl" />
+          <mesh filename="package://mycobot_description/meshes/stl/visual/link4.dae" />
         </geometry>
         <origin xyz="0 0 0" rpy="0 0 0" />
@@ -94,4 +97,5 @@
         <geometry>
           <mesh filename="package://mycobot_description/meshes/stl/collision/link4.stl" />
+          <!-- <mesh filename="package://mycobot_description/meshes/stl/visual/link4.stl" /> -->
         </geometry>
         <origin xyz="0 0 0" rpy="0 0 0" />
@@ -106,5 +110,5 @@
       <visual>
         <geometry>
-          <mesh filename="package://mycobot_description/meshes/stl/visual/link5.stl" />
+          <mesh filename="package://mycobot_description/meshes/stl/visual/link5.dae" />
         </geometry>
         <origin xyz="0 0 0" rpy="0 0 0" />
@@ -114,4 +118,5 @@
         <geometry>
           <mesh filename="package://mycobot_description/meshes/stl/collision/link5.stl" />
+          <!-- <mesh filename="package://mycobot_description/meshes/stl/visual/link5.stl" /> -->
         </geometry>
         <origin xyz="0 0 0" rpy="0 0 0" />
@@ -126,5 +131,5 @@
       <visual>
         <geometry>
-          <mesh filename="package://mycobot_description/meshes/stl/visual/link6.stl" />
+          <mesh filename="package://mycobot_description/meshes/stl/visual/link6.dae" />
         </geometry>
         <origin xyz="0 0 0 " rpy="0 0 0" />
@@ -134,4 +139,5 @@
         <geometry>
           <mesh filename="package://mycobot_description/meshes/stl/collision/link6.stl" />
+          <!-- <mesh filename="package://mycobot_description/meshes/stl/visual/link6.stl" /> -->
         </geometry>
         <origin xyz="0 0 0" rpy="0 0 0" />
@@ -146,14 +152,14 @@
       <visual>
         <geometry>
-          <cylinder length="0.005" radius="0.02" />
-        </geometry>
-        <origin xyz="0 0.0025 0" rpy="${M_PI/2} 0 0" />
-        <material name="green" />
-      </visual>
-      <collision>
-        <geometry>
-          <cylinder length="0.005" radius="0.02" />
-        </geometry>
-        <origin xyz="0 0.0025 0" rpy="${M_PI/2} 0 0" />
+          <mesh filename="package://mycobot_description/meshes/stl/visual/link7.dae" />
+        </geometry>
+        <origin xyz="0 0 0 " rpy="0 0 0" />
+        <material name="white" />
+      </visual>
+      <collision>
+        <geometry>
+          <mesh filename="package://mycobot_description/meshes/stl/collision/link7.stl" />
+        </geometry>
+        <origin xyz="0 0 0" rpy="0 0 0" />
       </collision>
       <inertial>
@@ -204,9 +210,9 @@
     </joint>
     <joint name="${mycobot_joint_6}" type="revolute">
-      <axis xyz="0 1 0" />
+      <axis xyz="0 0 1" />
       <limit effort="10.0" lower="-${M_PI}" upper="${M_PI}" velocity="${joint_velocity_limit}" />
       <parent link="${mycobot_link_6}" />
       <child link="${mycobot_link_7}" />
-      <origin xyz="0 0.0456 0.03792" rpy="0 0 0" />
+      <origin xyz="0 0.0351 0.03792" rpy="${-M_PI/2} 0 0" />
       <dynamics damping="1.0e-6" friction="2.0e-1" />
     </joint>
